Commit message: The correct mesh is now loaded. Packages is tested on ros-noetic

File: xacro/urg-04lx.xacro (robot description, xacro)
@@ -11,5 +11,5 @@
         <origin xyz="0 0 0" rpy="0 0 0"/>
         <geometry>
-          <mesh filename="package://urdf_tutorial/meshes/hokuyo.dae"/>
+          <mesh filename="package://ros_hokuyo_urg04lx_description/meshes/hokuyo.dae"/>
         </geometry>
       </visual>
